File: SPM-STMTB-V1.kicad_sch (KiCad schematic)
At the start: 34 parts, among them J1 Conn_01x13_Pin, J2 Conn_01x15_Pin, J3 Conn_01x08_Pin, U1 LD1117S33TR_SOT223, U2 TLP185, U3 STM32C092KBT6, U6 74LVC1G14, Y1 Resonator

Commit message: PTr電流制限抵抗の変更
Parts:
- R2: value R4.7k -> R1k
Changed lines of the file:
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@@
 			)
 		)
-		(property "Value" "R4.7k"
+		(property "Value" "R1k"
 			(at 34.036 164.592 0)
 			(effects
